File: TTL_to_HDMI.kicad_sch (KiCad schematic)
At the start: 62 parts, among them J1 HDMI_A_1.4, J2 Conn_01x19_Female, J3 Conn_01x19_Female, U1 1x50, U2 1x50, U3 TFP410PAP, U4 MT3420C

Commit message: Upload_V3 V4 and PDF V3
Parts:
- removed C1, C10, C12, C5, C6, C9: 4µ7, Capacitor_SMD:C_0603_1608Metric, symbol Device:C
- removed C11, C2: 100n, Capacitor_SMD:C_0603_1608Metric, symbol Device:C
- removed D1: LED, Capacitor_SMD:C_0805_2012Metric, symbol Device:LED
- removed J1: HDMI_A_1.4, Connector_HDMI:HDMI_A_Molex_208658-1001_Horizontal, symbol Connector:HDMI_A_1.4
- removed J2, J3: Conn_01x19_Female, Connector_FFC-FPC:Hirose_FH12-19S-0.5SH_1x19-1MP_P0.50mm_Horizontal, symbol Connector:Conn_01x19_Female
- removed L1: 2µ2, Inductor_SMD:L_TDK_NLV32_3.2x2.5mm, symbol Device:L
- removed R22: 510, Resistor_SMD:R_0603_1608Metric, symbol Device:R
- removed R24, R25, R35, R37, R38, R39, R40: 5K, Resistor_SMD:R_0603_1608Metric, symbol Device:R
- removed R26: 0, Resistor_SMD:R_0603_1608Metric, symbol Device:R
- removed R27, R28, R29, R30, R31, R32, R33, R34: 10, Resistor_SMD:R_0603_1608Metric, symbol Device:R
- removed R36: 10K, Resistor_SMD:R_0603_1608Metric, symbol Device:R
- removed R41: 450K, Resistor_SMD:R_0603_1608Metric, symbol Device:R
- removed R42: 100K, Resistor_SMD:R_0603_1608Metric, symbol Device:R
- removed U3: TFP410PAP, Package_QFP:HTQFP-64-1EP_10x10mm_P0.5mm_EP8x8mm_Mask4.4x4.4mm_ThermalVias, symbol Video:TFP410PAP
- removed U4: MT3420C, Package_TO_SOT_SMD:SOT-23-6, symbol TheBrutzlers_Lib:MT3420C-mt3420c
- added J1, J2: Conn_01x32_Pin, Connector_FFC-FPC:Hirose_FH12-32S-0.5SH_1x32-1MP_P0.50mm_Horizontal, symbol Connector:Conn_01x32_Pin
- added Q2: Q_NPN_BEC, Package_TO_SOT_SMD:SOT-23, symbol Device:Q_NPN_BEC
- added U3, U6, U7, U8: 74LVX541, Package_SO:TSSOP-20_4.4x6.5mm_P0.65mm, symbol 74xx:74HCT541
- added U5: NANO_9K, TheBrutzlers_Lib:Nano 9K, symbol TheBrutzlers_Lib:NANO_9K
- R1, R10, R13, R15, R17, R18, R21, R5, R7: value 5K -> 10K
- R11: now not fitted
- R12, R14, R16, R19, R20, R3, R6, R8, R9: value 5K -> 10K; NP NP -> (none); now in the parts list
- R2: value 5K -> 100K; NP NP -> (none); now in the parts list
- R4: value 5K -> 0; now not fitted
Connections:
- net +3V3: now also J1.11 (Pin_11), J2.22 (Pin_22), U3.20 (VCC), U5.25 (3V3), U6.20 (VCC), U7.20 (VCC), U8.20 (VCC); no longer R1.1, R12.1, R14.1, R16.1, R18.1, R20.1, R5.1, R7.1, R9.1
- net +5V: now also R4.2, J1.13 (Pin_13), J2.20 (Pin_20), U5.31 (5V); no longer U1.1, U1.2, U2.49, U2.50
- net B0: now also U6.4 (A2)
- net B1: now also U6.3 (A1)
- net B2: now also U6.2 (A0)
- net B3: now also U3.9 (A7)
- net B4: now also U3.8 (A6)
- net B5: now also U3.7 (A5)
- net B6: now also U3.6 (A4)
- net B7: now also U3.5 (A3)
- net CLK: now also U8.5 (A3)
- net G0: now also U7.4 (A2)
- net G1: now also U7.3 (A1)
- net G2: now also U7.2 (A0)
- net G3: now also U6.9 (A7)
- net G4: now also U6.8 (A6)
- net G5: now also U6.7 (A5)
- net G6: now also U6.6 (A4)
- net G7: now also U6.5 (A3)
- net GND: now also R14.1, R15.1, R16.1, R17.1, R18.1, R19.1, R20.1, R21.1, J1.14 (Pin_14), J2.19 (Pin_19), Q2.2 (E), U3.10 (GND), U5.26 (GND), U6.10 (GND), U7.10 (GND), U8.10 (GND), U8.6 (A4), U8.7 (A5), U8.8 (A6), U8.9 (A7); no longer R10.2, R13.2, R15.2, R17.2, R19.2, R21.2, R4.2, R6.2, R8.2
- net R0: now also U8.4 (A2)
- net R1: now also U8.3 (A1)
- net R2: now also U8.2 (A0)
- net R3: now also U7.9 (A7)
- net R4: now also U7.8 (A6)
- net R5: now also U7.7 (A5)
- net R6: now also U7.6 (A4)
- net R7: now also U7.5 (A3)
- net VS: now reaches U1.10, U2.41
- net VS: now also U3.3 (A1)
- net HS: now reaches U1.11, U2.40
- net HS: now also U3.4 (A2)
- net DE: now reaches U1.9, U2.42
- net DE: now also U3.2 (A0)
- net CTL1 renamed 25
- net 25: now also R20.2, J1.8 (Pin_8), J2.25 (Pin_25), U5.41 (IOT12A); no longer R13.1
- net CTL2 renamed 31
- net 31: now also R5.2, J1.2 (Pin_2), J2.31 (Pin_31), U5.47 (IOT8A); no longer R15.1
- net CTL3 renamed 29
- net 29: now also R7.2, J1.4 (Pin_4), J2.29 (Pin_29), U5.45 (IOT10A); no longer R17.1
- net DKEN: no longer names the net of R4.1
- net DKEN: now also U1.1, U1.2, U2.49, U2.50; no longer R3.2
- net EDGE: no longer names the net of R2.1
- net EDGE: now also R1.1, Q2.1 (B); no longer R1.2
- net MSEN renamed F_B1
- net F_B1: now also U6.17 (Y1); no longer R5.2
- net SCL renamed 27
- net 27: now also R9.2, J1.6 (Pin_6), J2.27 (Pin_27), U5.43 (IOT11A); no longer R19.1
- removed net SDA: R20.2, R21.1
- net nPD renamed F_R2
- net F_R2: now also U8.18 (Y0); no longer R7.2
- net nRST renamed F_R0
- net F_R0: now also U8.16 (Y2); no longer R9.2
- new net 24: J1.9 (Pin_9), J2.24 (Pin_24), R13.2, R21.2, U5.40 (IOT12B)
- new net 26: J1.7 (Pin_7), J2.26 (Pin_26), R10.2, R19.2, U5.42 (IOT11B)
- new net 28: J1.5 (Pin_5), J2.28 (Pin_28), R17.2, R8.2, U5.44 (IOT10B)
- new net 30: J1.3 (Pin_3), J2.30 (Pin_30), R15.2, R6.2, U5.46 (IOT8B)
- new net 32: J1.1 (Pin_1), J2.32 (Pin_32), R1.2, U5.48 (IOR5A)
- new net F_B0: R7.1, U6.16 (Y2)
- new net F_B2: R5.1, U6.18 (Y0)
- new net F_B3: J1.24 (Pin_24), J2.9 (Pin_9), U3.11 (Y7), U5.10 (IOB13B)
- new net F_B4: J1.25 (Pin_25), J2.8 (Pin_8), U3.12 (Y6), U5.9 (IOB13A)
- new net F_B5: J1.26 (Pin_26), J2.7 (Pin_7), U3.13 (Y5), U5.8 (IOB11B)
- new net F_B6: J1.27 (Pin_27), J2.6 (Pin_6), U3.14 (Y4), U5.7 (IOB11A)
- new net F_B7: J1.28 (Pin_28), J2.5 (Pin_5), U3.15 (Y3), U5.6 (IOB8B)
- new net F_CLK: J1.18 (Pin_18), J2.15 (Pin_15), U5.14 (IOB29A), U8.15 (Y3)
- new net F_DE: J1.32 (Pin_32), J2.1 (Pin_1), U3.18 (Y0), U5.1 (IOB31B)
- new net F_G0: R13.1, U7.16 (Y2)
- new net F_G1: R12.1, U7.17 (Y1)
- new net F_G2: J1.12 (Pin_12), J2.21 (Pin_21), U5.30 (IOR24B), U7.18 (Y0)
- new net F_G3: J1.16 (Pin_16), J2.17 (Pin_17), U5.38 (IOT37B), U6.11 (Y7)
- new net F_G4: J1.15 (Pin_15), J2.18 (Pin_18), U5.22 (IOR13A), U6.12 (Y6)
- new net F_G5: J1.22 (Pin_22), J2.11 (Pin_11), U5.18 (IOR15B), U6.13 (Y5)
- new net F_G6: J1.21 (Pin_21), J2.12 (Pin_12), U5.17 (IOR17B), U6.14 (Y4)
- new net F_G7: J1.20 (Pin_20), J2.13 (Pin_13), U5.16 (IOB41B), U6.15 (Y3)
- new net F_HS: J1.30 (Pin_30), J2.3 (Pin_3), U3.16 (Y2), U5.3 (IOB29B)
- new net F_OE1: Q2.3 (C), R3.2, U3.1 (G1), U3.19 (G2), U6.1 (G1), U6.19 (G2), U7.1 (G1), U7.19 (G2), U8.1 (G1), U8.19 (G2)
- new net F_R1: R9.1, U8.17 (Y1)
- new net F_R3: J1.19 (Pin_19), J2.14 (Pin_14), U5.15 (IOB41A), U7.11 (Y7)
- new net F_R4: J1.10 (Pin_10), J2.23 (Pin_23), U5.39 (IOT37A), U7.12 (Y6)
- new net F_R5: J1.29 (Pin_29), J2.4 (Pin_4), U5.4 (IOB33A), U7.13 (Y5)
- new net F_R6: J1.17 (Pin_17), J2.16 (Pin_16), U5.12 (IOB23B), U7.14 (Y4)
- new net F_R7: J1.23 (Pin_23), J2.10 (Pin_10), U5.11 (IOB23A), U7.15 (Y3)
- new net F_VS: J1.31 (Pin_31), J2.2 (Pin_2), U3.17 (Y1), U5.2 (IOB31A)
Other:
- note removed: "24 Bit = HIGH 12 Bit = LOW"
- note removed: "600mV"
- company: (none) -> theBrutzler
- title: (none) -> TTL->HDMI R1gol
