File: TTL_to_HDMI.kicad_sch (KiCad schematic)
At the start: 35 parts, among them J1 Conn_01x32_Pin, J2 Conn_01x32_Pin, Q2 Q_NPN_BEC, U1 1x50, U2 1x50, U3 74LVX541, U5 NANO_9K, U6 74LVX541, U7 74LVX541, U8 74LVX541

Commit message: Update Final stade
Parts:
- removed J1, J2: Conn_01x32_Pin, Connector_FFC-FPC:Hirose_FH12-32S-0.5SH_1x32-1MP_P0.50mm_Horizontal, symbol Connector:Conn_01x32_Pin
- removed R1, R10, R12, R13, R3, R5, R6, R7, R8, R9: 10K, Resistor_SMD:R_0603_1608Metric, symbol Device:R
- removed R11, R4: 0, Resistor_SMD:R_0603_1608Metric, symbol Device:R
- removed U3, U6, U7, U8: 74LVX541, Package_SO:TSSOP-20_4.4x6.5mm_P0.65mm, symbol 74xx:74HCT541
- added C14, C15, C16: 10u, Capacitor_SMD:C_0603_1608Metric, symbol Device:C
- added C5, C6: 100n, Capacitor_SMD:C_0603_1608Metric, symbol Device:C
- added J1: Conn_01x02_Socket, Connector_PinHeader_2.54mm:PinHeader_1x02_P2.54mm_Vertical, symbol Connector:Conn_01x02_Socket
- added J2: ONLY DUMMY, Connector_PinHeader_2.54mm:PinHeader_2x09_P2.54mm_Vertical, symbol Connector_Generic:Conn_02x08_Counter_Clockwise
- added J3, J5: Conn_01x35_Pin, Connector_FFC-FPC:Amphenol_F32Q-1A7x1-11035_1x35-1MP_P0.5mm_Horizontal, symbol Connector:Conn_01x35_Pin
- added R22, R23, R24, R25, R26, R27, R28, R29, R30, R31, R32, R33: 1K, Resistor_SMD:R_0603_1608Metric, symbol Device:R
- added U4, U6, U7, U8: 74HC245, Package_SO:TSSOP-20_4.4x6.5mm_P0.65mm, symbol 74xx:74HC245
- C3, C4, C7, C8: LCSC (none) -> C6119883
- R14, R15, R16, R17, R18, R19, R20, R21: value 10K -> 1K; LCSC (none) -> C54920984
- R2: LCSC (none) -> C54920958
- U1, U2: LCSC (none) -> C22459571
- U5: LCSC (none) -> DNP; now not fitted; now left out of the parts list
Connections:
- net +3V3: now also C14.1, C15.1, C5.2, J3.5 (Pin_5), J5.31 (Pin_31), R31.1, R33.1, U4.20 (VCC), U6.20 (VCC), U7.20 (VCC), U8.20 (VCC)
- net +5V: now also C16.1, C6.2, J1.2 (Pin_2)
- net B0: now also U1.32, U2.19, U7.7 (A5); no longer U1.19, U2.32
- net B1: now also U1.33, U2.18, U7.8 (A6); no longer U1.18, U2.33
- net B2: now also U1.34, U2.17, U7.9 (A7); no longer U1.17, U2.34
- net B3: now also U1.35, U2.16, U4.2 (A0); no longer U1.16, U2.35
- net B4: now also U1.36, U2.15, U4.3 (A1); no longer U1.15, U2.36
- net B5: now also U1.37, U2.14, U4.4 (A2); no longer U1.14, U2.37
- net B6: now also U1.38, U2.13, U4.5 (A3); no longer U1.13, U2.38
- net B7: now also U1.39, U2.12, U4.6 (A4); no longer U1.12, U2.39
- net CLK: now also U1.14, U2.37, U8.3 (A1); no longer U1.37, U2.14
- net DE: now also U1.42, U2.9, U4.9 (A7); no longer U1.9, U2.42
- net F_B0: now also U5.7 (IOB11A), J3.23 (Pin_23), J5.13 (Pin_13), U7.13 (B5)
- net F_B1: now also U5.8 (IOB11B), J3.24 (Pin_24), J5.12 (Pin_12), U7.12 (B6)
- net F_B2: now also U5.9 (IOB13A), J3.25 (Pin_25), J5.11 (Pin_11), U7.11 (B7)
- net F_B3: now also J3.26 (Pin_26), J5.10 (Pin_10), U4.18 (B0)
- net F_B4: now also U5.11 (IOB23A), J3.27 (Pin_27), J5.9 (Pin_9), U4.17 (B1); no longer U5.9 (IOB13A)
- net F_B5: now also U5.12 (IOB23B), J3.28 (Pin_28), J5.8 (Pin_8), U4.16 (B2); no longer U5.8 (IOB11B)
- net F_B6: now also U5.14 (IOB29A), J3.29 (Pin_29), J5.7 (Pin_7), U4.15 (B3); no longer U5.7 (IOB11A)
- net F_B7: now also U5.15 (IOB41A), J3.30 (Pin_30), J5.6 (Pin_6), U4.14 (B4); no longer U5.6 (IOB8B)
- net F_CLK: now also U5.27 (IOB15B), J3.2 (Pin_2), J5.34 (Pin_34), U8.17 (B1); no longer U5.14 (IOB29A)
- net F_DE: now also U5.22 (IOR13A), J3.34 (Pin_34), J5.2 (Pin_2), U4.11 (B7); no longer U5.1 (IOB31B)
- net F_G0: now also R27.1, U6.13 (B5)
- net F_G1: now also R28.1, U6.12 (B6)
- net F_G2: now also R29.1, U6.11 (B7); no longer U5.30 (IOR24B)
- net F_G3: now also U5.1 (IOB31B), J3.18 (Pin_18), J5.18 (Pin_18), U7.18 (B0); no longer U5.38 (IOT37B)
- net F_G4: now also U5.2 (IOB31A), J3.19 (Pin_19), J5.17 (Pin_17), U7.17 (B1); no longer U5.22 (IOR13A)
- net F_G5: now also U5.3 (IOB29B), J3.20 (Pin_20), J5.16 (Pin_16), U7.16 (B2); no longer U5.18 (IOR15B)
- net F_G6: now also U5.4 (IOB33A), J3.21 (Pin_21), J5.15 (Pin_15), U7.15 (B3); no longer U5.17 (IOR17B)
- net F_G7: now also U5.6 (IOB8B), J3.22 (Pin_22), J5.14 (Pin_14), U7.14 (B4); no longer U5.16 (IOB41B)
- net F_HS: now also U5.17 (IOR17B), J3.32 (Pin_32), J5.4 (Pin_4), U4.13 (B5); no longer U5.3 (IOB29B)
- net F_R0: now also U5.30 (IOR24B), J3.7 (Pin_7), J5.29 (Pin_29), U8.13 (B5)
- net F_R1: now also U5.38 (IOT37B), J3.8 (Pin_8), J5.28 (Pin_28), U8.12 (B6)
- net F_R2: now also U5.39 (IOT37A), J3.9 (Pin_9), J5.27 (Pin_27), U8.11 (B7)
- net F_R3: now also R22.1, U6.18 (B0); no longer U5.15 (IOB41A)
- net F_R4: now also R23.1, U6.17 (B1); no longer U5.39 (IOT37A)
- net F_R5: now also R24.1, U6.16 (B2); no longer U5.4 (IOB33A)
- net F_R6: now also R25.1, U6.15 (B3); no longer U5.12 (IOB23B)
- net F_R7: now also R26.1, U6.14 (B4); no longer U5.11 (IOB23A)
- net F_VS: now also U5.18 (IOR15B), J3.33 (Pin_33), J5.3 (Pin_3), U4.12 (B6); no longer U5.2 (IOB31A)
- net G0: now also U1.24, U2.27, U6.7 (A5); no longer U1.27, U2.24
- net G1: now also U1.25, U2.26, U6.8 (A6); no longer U1.26, U2.25
- net G2: now also U1.26, U2.25, U6.9 (A7); no longer U1.25, U2.26
- net G3: now also U1.27, U2.24, U7.2 (A0); no longer U1.24, U2.27
- net G4: now also U1.28, U2.23, U7.3 (A1); no longer U1.23, U2.28
- net G5: now also U1.29, U2.22, U7.4 (A2); no longer U1.22, U2.29
- net G6: now also U1.30, U2.21, U7.5 (A3); no longer U1.21, U2.30
- net G7: now also U1.31, U2.20, U7.6 (A4); no longer U1.20, U2.31
- net GND: now also U1.13, U1.15, U1.3, U1.46, U2.36, U2.38, U2.48, U2.5, C14.2, C15.2, C16.2, C5.1, C6.1, J1.1 (Pin_1), J3.1 (Pin_1), J3.3 (Pin_3), J3.31 (Pin_31), J3.35 (Pin_35), J3.6 (Pin_6), J5.1 (Pin_1), J5.30 (Pin_30), J5.33 (Pin_33), J5.35 (Pin_35), J5.5 (Pin_5), R32.2, U4.10 (GND), U6.10 (GND), U7.10 (GND), U8.10 (GND), U8.2 (A0), U8.4 (A2), U8.5 (A3), U8.6 (A4); no longer U1.36, U1.38, U1.48, U1.5, U2.13, U2.15, U2.3, U2.46
- net HS: now also U1.40, U2.11, U4.7 (A5); no longer U1.11, U2.40
- net R0: now also U1.16, U2.35, U8.7 (A5); no longer U1.35, U2.16
- net R1: now also U1.17, U2.34, U8.8 (A6); no longer U1.34, U2.17
- net R2: now also U1.18, U2.33, U8.9 (A7); no longer U1.33, U2.18
- net R3: now also U1.19, U2.32, U6.2 (A0); no longer U1.32, U2.19
- net R4: now also U1.20, U2.31, U6.3 (A1); no longer U1.31, U2.20
- net R5: now also U1.21, U2.30, U6.4 (A2); no longer U1.30, U2.21
- net R6: now also U1.22, U2.29, U6.5 (A3); no longer U1.29, U2.22
- net R7: now also U1.23, U2.28, U6.6 (A4); no longer U1.28, U2.23
- net VS: now also U1.41, U2.10, U4.8 (A6); no longer U1.10, U2.41
- net at Q2.1 (B), R2.1: now also R30.1
- net at U1.1, U2.50: no longer U1.2, U2.49
- net V_BLK: now reaches U1.49, U2.2
- net V_BLK: now also U1.50, U2.1
- net 24 renamed 10
- net 10: now also R14.2, J3.10 (Pin_10), J5.26 (Pin_26), R22.2; no longer R21.2
- net 25 renamed 11
- net 11: now also R15.2, J3.11 (Pin_11), J5.25 (Pin_25), R23.2; no longer R20.2
- net 26 renamed 12
- net 12: now also R16.2, J3.12 (Pin_12), J5.24 (Pin_24), R24.2; no longer R19.2
- net 27 renamed 13
- net 13: now also R17.2, J3.13 (Pin_13), J5.23 (Pin_23), R25.2; no longer R18.2
- net 28 renamed 14
- net 14: now also R18.2, J3.14 (Pin_14), J5.22 (Pin_22), R26.2; no longer R17.2
- net 29 renamed 15
- net 15: now also R19.2, J3.15 (Pin_15), J5.21 (Pin_21), R27.2; no longer R16.2
- net 30 renamed 16
- net 16: now also R20.2, J3.16 (Pin_16), J5.20 (Pin_20), R28.2; no longer R15.2
- net 31 renamed 17
- net 17: now also R21.2, J3.17 (Pin_17), J5.19 (Pin_19), R29.2; no longer R14.2
- net 32 renamed 4
- net 4: now also J3.4 (Pin_4), J5.32 (Pin_32), R30.2
- net F_OE1 renamed F_OE
- net F_OE: now also R31.2, U4.19 (CE), U6.19 (CE), U7.19 (CE), U8.19 (CE)
- net VCC: no longer names the net of U1.7, U2.44
- new net: U1.10, U2.41
- new net: U1.11, U2.40
- new net: U1.12, U2.39
- new net: U1.2, U2.49
- new net: U1.48, U2.3
- new net: U1.5, U2.46
- new net: U1.9, U2.42
- new net F_DIR: R32.1, R33.2, U4.1 (A->B), U6.1 (A->B), U7.1 (A->B), U8.1 (A->B)
- no-connect marks 0 -> 32
Other:
- moved on the sheet: Q2, R14, R2, U1
